File: Keyboard_Prototyping.kicad_pcb (KiCad board)
At the start: 2 copper layers, 39 x 70 mm, 21 parts, among them J1 Conn_02x03_Odd_Even, J18 Conn_02x03_Odd_Even, J2 Conn_02x03_Odd_Even, J3 Conn_02x03_Odd_Even, J4 Conn_02x03_Odd_Even, J5 Conn_01x08, J6 Conn_02x03_Odd_Even, J7 Conn_02x03_Odd_Even, J8 Conn_02x03_Odd_Even, SW1 A, SW2 C, SW3 B, SW4 D

Commit message: Generated fabrication files
Other:
- board text added: "Brett Hallen, Aug 2025 Port Macquarie, Australia www.youtube.com/@Brfff"
- board text added: "Cherry MX Switch A"
- board text added: "Cherry MX Switch B"
- board text added: "Cherry MX Switch C"
- board text added: "Cherry MX Switch D"
Changed lines of the file:
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@@
 	(paper "A5")
 	(title_block
-		(title "Keyboard Prototyper")
+		(title "Keyboard Prototyping Board")
 		(date "6/Aug/2025")
 		(rev "A")
@@
 		(layer "Edge.Cuts")
 	)
+	(gr_text "Cherry MX\nSwitch D"
+		(at 62.17 99.55 0)
+		(layer "F.SilkS")
+		(effects
+			(font
+				(size 1 1)
+				(thickness 0.1)
+			)
+			(justify bottom)
+		)
+	)
+	(gr_text "Cherry MX\nSwitch B"
+		(at 43.17 99.55 0)
+		(layer "F.SilkS")
+		(effects
+			(font
+				(size 1 1)
+				(thickness 0.1)
+			)
+			(justify bottom)
+		)
+	)
+	(gr_text "Cherry MX\nSwitch C"
+		(at 62.17 80.55 0)
+		(layer "F.SilkS")
+		(effects
+			(font
+				(size 1 1)
+				(thickness 0.1)
+			)
+			(justify bottom)
+		)
+	)
+	(gr_text "Brett's Keyboard\nPrototyper"
+		(at 54.17 49.55 90)
+		(layer "F.SilkS")
+		(effects
+			(font
+				(size 1 1)
+				(thickness 0.1)
+			)
+			(justify bottom)
+		)
+	)
+	(gr_text "Cherry MX\nSwitch A"
+		(at 43.17 80.55 0)
+		(layer "F.SilkS")
+		(effects
+			(font
+				(size 1 1)
+				(thickness 0.1)
+			)
+			(justify bottom)
+		)
+	)
 	(gr_text "A  C\nB  D"
 		(at 53.09 63.84 0)
@@
 		)
 	)
-	(gr_text "Brett's Keyboard\nPrototyper"
-		(at 52.09 85.84 0)
+	(gr_text "Brett Hallen, Aug 2025\nPort Macquarie, Australia\nwww.youtube.com/@Brfff"
+		(at 62.17 85.55 0)
 		(layer "B.SilkS")
 		(effects
@@
 				(thickness 0.1)
 			)
-			(justify bottom mirror)
+			(justify left bottom mirror)
 		)
 	)
